File: hardware/SolderingStation.kicad_pcb (KiCad board)
At the start: 2 copper layers, 0 parts

Commit message: starting pcb
Parts:
- added BZ1: Buzzer, Buzzer_Beeper:Buzzer_12x9.5RM7.6, F.Cu at (204.8, 82.3)
- added C1: 0.1u, Capacitor_SMD:C_0603_1608Metric, F.Cu at (187.8, 76.8)
- added C10: 22pF, Capacitor_SMD:C_0603_1608Metric, F.Cu at (187.8, 81.8)
- added C11: 100uF, Capacitor_SMD:CP_Elec_6.3x5.4, F.Cu at (242.9, 108.9)
- added C12: 0.1u, Capacitor_SMD:C_0603_1608Metric, F.Cu at (235.5, 111.6)
- added C13: 10uF, Capacitor_SMD:CP_Elec_5x5.4, F.Cu at (242.1, 101.4)
- added C14: 22uF, Capacitor_Tantalum_SMD:CP_EIA-3216-18_Kemet-A, F.Cu at (230.6, 112.5)
- added C15: 0.1u, Capacitor_SMD:C_0603_1608Metric, F.Cu at (253.9, 67.6)
- added C16: 0.1u, Capacitor_SMD:C_0603_1608Metric, F.Cu at (187.8, 84.4)
- added C17: 0.1u, Capacitor_SMD:C_0603_1608Metric, F.Cu at (187.8, 86.9)
- added C18: 0.1u, Capacitor_SMD:C_0603_1608Metric, F.Cu at (187.8, 89.4)
- added C19: 0.1u, Capacitor_SMD:C_0603_1608Metric, F.Cu at (187.8, 91.9)
- added C2: 0.1u, Capacitor_SMD:C_0603_1608Metric, F.Cu at (235.5, 109.1)
- added C20: 0.1u, Capacitor_SMD:C_0603_1608Metric, F.Cu at (191.8, 76.8)
- added C3: 10uF, Capacitor_SMD:CP_Elec_5x5.4, F.Cu at (242.1, 94.6)
- added C4: 10uF 50V, Capacitor_SMD:C_1206_3216Metric, F.Cu at (263.8, 105.6)
- added C5: 1u, Capacitor_SMD:C_0603_1608Metric, F.Cu at (253.9, 60.1)
- added C6: 0.1u, Capacitor_SMD:C_0603_1608Metric, F.Cu at (253.9, 62.6)
- added C7: 0.1u, Capacitor_SMD:C_0603_1608Metric, F.Cu at (253.9, 65.1)
- added C8: 22uF, Capacitor_Tantalum_SMD:CP_EIA-3216-18_Kemet-A, F.Cu at (230.6, 109.4)
- added C9: 22pF, Capacitor_SMD:C_0603_1608Metric, F.Cu at (187.8, 79.3)
- added D1: SS54, Diode_SMD:D_SMA, F.Cu at (244.0, 54.1)
- added D2: SS54, Diode_SMD:D_SMA, F.Cu at (265.1, 101.6)
- added D3: BZT52C12, Diode_SMD:D_SOD-123F, F.Cu at (265.2, 92.8)
- added D4: 1N4148, Diode_SMD:D_SOD-123F, B.Cu at (61.4, 132.0)
- added D5: BZT52C3V3, Diode_SMD:D_SOD-123F, F.Cu at (266.7, 60.5)
- added GX12: Soldering Iron, SolderingStationLib:GX-12-5, B.Cu at (132.0, 105.2)
- added GX16: Hot Air, SolderingStationLib:GX-16-8, B.Cu at (61.0, 106.0)
- added J1: AC Screw Terminal, TerminalBlock:TerminalBlock_MaiXu_MX126-5.0-03P_1x03_P5.00mm, F.Cu at (210.8, 38.2)
- added J10: Power, TerminalBlock:TerminalBlock_MaiXu_MX126-5.0-03P_1x03_P5.00mm, F.Cu at (51.0, 127.0)
- added J11: Logic, Connector_PinHeader_2.54mm:PinHeader_1x02_P2.54mm_Vertical, F.Cu at (68.0, 137.0)
- added J12: SWD, Connector_PinHeader_2.54mm:PinHeader_1x04_P2.54mm_Vertical, F.Cu at (223.5, 56.5)
- added J13: Relay Contact, TerminalBlock:TerminalBlock_MaiXu_MX126-5.0-02P_1x02_P5.00mm, F.Cu at (97.0, 139.0)
- added J14: Relay Coil, TerminalBlock:TerminalBlock_MaiXu_MX126-5.0-02P_1x02_P5.00mm, F.Cu at (65.0, 128.0)
- added J2: Iron Encoder, Connector_PinHeader_2.54mm:PinHeader_1x05_P2.54mm_Vertical, F.Cu at (135.0, 65.2)
- added J3: Hot Air Encoder, Connector_PinHeader_2.54mm:PinHeader_1x05_P2.54mm_Vertical, F.Cu at (55.0, 55.0)
- added J4: OLED, Connector_PinHeader_2.54mm:PinHeader_1x04_P2.54mm_Vertical, F.Cu at (98.5, 48.0)
- added J5: High Voltage, TerminalBlock:TerminalBlock_MaiXu_MX126-5.0-02P_1x02_P5.00mm, F.Cu at (89.0, 125.0)
- added J6: UART, Connector_PinHeader_2.54mm:PinHeader_1x04_P2.54mm_Vertical, F.Cu at (218.9, 56.5)
- added J7: STM BOOT, Connector_PinHeader_2.54mm:PinHeader_1x03_P2.54mm_Vertical, F.Cu at (221.6, 45.6)
- added J8: +5V, TerminalBlock:TerminalBlock_MaiXu_MX126-5.0-02P_1x02_P5.00mm, F.Cu at (210.8, 48.3)
- added J9: Logic, Connector_PinHeader_2.54mm:PinHeader_1x02_P2.54mm_Vertical, F.Cu at (214.3, 68.7)
- added JP1: Jumper_2_Open, Connector_PinHeader_2.54mm:PinHeader_1x03_P2.54mm_Vertical, F.Cu at (72.0, 130.5)
- added Q1: AOD4184, Package_TO_SOT_SMD:TO-252-2, F.Cu at (257.2, 95.3)
- added Q2: S8050, Package_TO_SOT_SMD:SOT-23-3, F.Cu at (265.0, 96.7)
- added Q3: S8050, Package_TO_SOT_SMD:SOT-23-3, B.Cu at (59.0, 137.1)
- added Q5: S8050, Package_TO_SOT_SMD:SOT-23-3, F.Cu at (198.9, 99.9)
- added Q6: 60T03H, Package_TO_SOT_SMD:TO-252-2, F.Cu at (234.7, 46.8)
- added Q7: BTA16-600B, Package_TO_SOT_THT:TO-220-3_Vertical, F.Cu at (231.0, 54.8)
- added R1: 300, Resistor_SMD:R_0603_1608Metric, F.Cu at (245.6, 34.4)
- added R10: 3k, Resistor_THT:R_Axial_DIN0207_L6.3mm_D2.5mm_P7.62mm_Horizontal, F.Cu at (251.8, 101.4)
- added R11: 2.2k, Resistor_SMD:R_0603_1608Metric, F.Cu at (263.0, 108.5)
- added R12: 1k, Resistor_SMD:R_0603_1608Metric, F.Cu at (191.8, 84.4)
- added R13: 10k, Resistor_SMD:R_0603_1608Metric, F.Cu at (191.8, 86.9)
- added R14: 10k, Resistor_SMD:R_0603_1608Metric, F.Cu at (191.8, 89.4)
- added R15: 1k, Resistor_SMD:R_0603_1608Metric, F.Cu at (191.8, 91.9)
- added R16: 3k, Resistor_THT:R_Axial_DIN0207_L6.3mm_D2.5mm_P7.62mm_Horizontal, F.Cu at (251.8, 105.4)
- added R17: 1k, Resistor_SMD:R_0603_1608Metric, F.Cu at (195.8, 76.8)
- added R18: 1k, Resistor_SMD:R_0603_1608Metric, F.Cu at (195.8, 79.3)
- added R19: 1k, Resistor_SMD:R_0603_1608Metric, F.Cu at (195.8, 81.8)
- added R2: 10k, Resistor_SMD:R_0603_1608Metric, F.Cu at (245.6, 36.9)
- added R20: 1k, Resistor_SMD:R_0603_1608Metric, F.Cu at (253.9, 70.1)
- added R21: 10k, Resistor_SMD:R_0603_1608Metric, F.Cu at (257.9, 60.1)
- added R22: 1k, Resistor_SMD:R_0603_1608Metric, F.Cu at (257.9, 62.6)
- added R23: 1k, Resistor_SMD:R_0603_1608Metric, F.Cu at (257.9, 65.1)
- added R24: 100k, Resistor_SMD:R_0603_1608Metric, F.Cu at (257.9, 67.6)
- added R25: 200k, Resistor_SMD:R_0603_1608Metric, F.Cu at (257.9, 70.1)
- added R26: 10k, Resistor_SMD:R_0603_1608Metric, F.Cu at (261.9, 60.1)
- added R27: 100k, Resistor_SMD:R_0603_1608Metric, F.Cu at (261.9, 62.6)
- added R28: 10k, Resistor_SMD:R_0603_1608Metric, F.Cu at (261.9, 65.1)
- added R29: 1k, Resistor_SMD:R_0603_1608Metric, F.Cu at (195.8, 84.4)
- added R3: 300, Resistor_SMD:R_0603_1608Metric, F.Cu at (245.6, 39.4)
- added R30: 1k, Resistor_SMD:R_0603_1608Metric, F.Cu at (195.8, 86.9)
- added R31: 1k, Resistor_SMD:R_0603_1608Metric, F.Cu at (195.8, 89.4)
- added R32: 1k, Resistor_SMD:R_0603_1608Metric, F.Cu at (195.8, 91.9)
- added R33: 1k, Resistor_SMD:R_0603_1608Metric, F.Cu at (199.8, 76.8)
- added R34: 1k, Resistor_SMD:R_0603_1608Metric, F.Cu at (199.8, 79.3)
- added R35: 1k, Resistor_SMD:R_0603_1608Metric, F.Cu at (199.8, 81.8)
- added R36: 10k, Resistor_SMD:R_0603_1608Metric, F.Cu at (199.8, 84.4)
- added R37: 10k, Resistor_SMD:R_0603_1608Metric, F.Cu at (199.8, 86.9)
- added R4: 390/0.5W, Resistor_THT:R_Axial_DIN0309_L9.0mm_D3.2mm_P12.70mm_Horizontal, F.Cu at (229.3, 35.5)
- added R5: 390/0.5W, Resistor_THT:R_Axial_DIN0309_L9.0mm_D3.2mm_P12.70mm_Horizontal, F.Cu at (229.3, 40.3)
- added R6: 10k, Resistor_SMD:R_0603_1608Metric, F.Cu at (191.8, 79.3)
- added R7: 10k, Resistor_SMD:R_0603_1608Metric, F.Cu at (191.8, 81.8)
- added R8: 10k, Resistor_SMD:R_0603_1608Metric, B.Cu at (54.2, 138.8)
- added R9: 10k, Resistor_SMD:R_0603_1608Metric, F.Cu at (72.0, 136.2)
- added SW1: SW_SPST, Button_Switch_THT:SW_PUSH_6mm_H8mm, F.Cu at (187.8, 95.2)
- added SW2: SW_SPST, TerminalBlock:TerminalBlock_MaiXu_MX126-5.0-02P_1x02_P5.00mm, F.Cu at (84.0, 139.0)
- added SW3: SW_SPST, Connector_PinHeader_2.54mm:PinHeader_1x02_P2.54mm_Vertical, F.Cu at (63.0, 137.0)
- added U1: MOC3063M, Package_DIP:DIP-6_W7.62mm_LongPads, F.Cu at (241.9, 44.7)
- added U2: AMS1117-3.3, Package_TO_SOT_SMD:SOT-223-3_TabPin2, F.Cu at (232.7, 95.4)
- added U4: AMS1117-3.3, Package_TO_SOT_SMD:SOT-223-3_TabPin2, F.Cu at (232.7, 103.7)
- added U5: STM32F103C8Tx, Package_QFP:LQFP-48_7x7mm_P0.5mm, F.Cu at (207.5, 94.8)
- added U6: MCP6002-xSN, Package_SO:SOIC-8_3.9x4.9mm_P1.27mm, F.Cu at (256.1, 74.7)
- added U7: ADS1115, Package_SO:MSOP-10_3x3mm_P0.5mm, F.Cu at (264.0, 73.7)
- added Y2: Crystal_GND24_Small, Crystal:Crystal_SMD_3225-4Pin_3.2x2.5mm, F.Cu at (198.9, 95.4)
Routing:
- net /Safety Relay/INPUT: track 0.00 -> 67.7 mm
- net /Safety Relay/OUTPUT: track 0.00 -> 59.7 mm
- net Net-(D4-A): track 0.00 -> 25.4 mm, vias 0 -> 2
- net /Safety Relay/24V: track 0.00 -> 22.8 mm
- net /Safety Relay/RELAY_CTRL: track 0.00 -> 17.8 mm
- net /Safety Relay/3V3: track 0.00 -> 14.1 mm
- net /Safety Relay/START_SENSE: track 0.00 -> 13.9 mm
- net GNDREF: track 0.00 -> 11.7 mm
- added copper zone on B.Cu, net GNDREF
- added copper zone on F.Cu, net GNDREF
Other:
- board outline added: 100 x 100 mm
