File: hardware/SolderingStation.kicad_sch (KiCad schematic)
At the start: 11 parts, among them J1 AC Screw Terminal, J12 SWD, J2 Iron Encoder, J3 Hot Air Encoder, J4 OLED, J6 UART, J7 STM BOOT, J8 +5V, J9 Logic

Commit message: fast commit
Connections:
- net COIL: now also GX16.3; no longer GX16.2
- net NEUTRAL: now also GX16.2; no longer GX16.3
Changed lines of the file:
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@@
 		)
 	)
-	(label "COIL"
+	(label "NEUTRAL"
 		(at 57.15 59.69 0)
 		(effects
@@
 		)
 	)
-	(label "NEUTRAL"
+	(label "COIL"
 		(at 57.15 62.23 0)
 		(effects

Commit message: pcb mvp
Parts:
- J8: footprint TerminalBlock:TerminalBlock_MaiXu_MX126-5.0-02P_1x02_P5.00mm -> TerminalBlock:TerminalBlock_MaiXu_MX126-5.0-03P_1x03_P5.00mm; symbol Connector:Screw_Terminal_01x02 -> Connector:Screw_Terminal_01x03
Connections:
- net 5V: now also J8.2 (Pin_2); no longer J8.1 (Pin_1)
- net COIL: now also GX16.2; no longer GX16.3
- net GNDREF: now also J8.3 (Pin_3); no longer J8.2 (Pin_2)
- net NEUTRAL: now also GX16.3, J1.3 (Pin_3); no longer GX16.2, J1.2 (Pin_2)
- net PE: now also J1.1 (Pin_1); no longer J1.3 (Pin_3)
- net ~220: now also J1.2 (Pin_2); no longer J1.1 (Pin_1)
- new net 24V: J8.1 (Pin_1)

Commit message: last
Parts:
- added D7, D8: LED, LED_SMD:LED_0805_2012Metric_Pad1.15x1.40mm_HandSolder, symbol Device:LED
- added R39: 2.2k, Resistor_SMD:R_0805_2012Metric_Pad1.20x1.40mm_HandSolder, symbol Device:R
- added R40: 10k, Resistor_SMD:R_0805_2012Metric_Pad1.20x1.40mm_HandSolder, symbol Device:R
Connections:
- net 24V: now also D8.2 (A)
- net 5V: now also D7.2 (A)
- net GNDREF: now also R39.1, R40.2
- new net: D8.1 (K), R40.1
- new net: D7.1 (K), R39.2
