File: hardware/heaterSwitch.kicad_sch (KiCad schematic)
At the start: 9 parts, among them Q1 AOD4184, Q2 S8050

Commit message: mvp
features:
	Logic Power Supply
	Safety Relay
	Main Unit
Parts:
- removed R15: 10k, symbol Device:R
Changed lines of the file:
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@@
 	(title_block
 		(title "Heater High side switch")
-		(date "2026-01-22")
-		(rev "vJun2026")
+		(date "2026-02-19")
+		(rev "vFeb2026")
 		(company "Author: Field Effect Transistor")
 		(comment 1 "https://github.com/Field-Effect-Transistor")
@@
 	)
 	(junction
-		(at 81.28 73.66)
-		(diameter 0)
-		(color 0 0 0 0)
-	)
-	(junction
 		(at 121.92 83.82)
 		(diameter 0)
@@
 	(wire
 		(pts
+			(xy 135.89 91.44) (xy 135.89 90.17)
+		)
+		(stroke
+			(width 0)
+			(type default)
+		)
+	)
+	(wire
+		(pts
 			(xy 121.92 58.42) (xy 124.46 58.42)
 		)
@@
 	(wire
 		(pts
-			(xy 76.2 73.66) (xy 81.28 73.66)
+			(xy 76.2 73.66) (xy 86.36 73.66)
 		)
 		(stroke
@@
 	(wire
 		(pts
-			(xy 81.28 58.42) (xy 81.28 63.5)
-		)
-		(stroke
-			(width 0)
-			(type default)
-		)
-	)
-	(wire
-		(pts
 			(xy 121.92 78.74) (xy 121.92 83.82)
 		)
@@
 	(wire
 		(pts
-			(xy 81.28 73.66) (xy 86.36 73.66)
-		)
-		(stroke
-			(width 0)
-			(type default)
-		)
-	)
-	(wire
-		(pts
 			(xy 111.76 58.42) (xy 121.92 58.42)
 		)
@@
 	(wire
 		(pts
+			(xy 135.89 90.17) (xy 139.7 90.17)
+		)
+		(stroke
+			(width 0)
+			(type default)
+		)
+	)
+	(wire
+		(pts
 			(xy 111.76 66.04) (xy 111.76 68.58)
 		)
@@
 	(wire
 		(pts
-			(xy 81.28 71.12) (xy 81.28 73.66)
-		)
-		(stroke
-			(width 0)
-			(type default)
-		)
-	)
-	(wire
-		(pts
 			(xy 101.6 50.8) (xy 96.52 50.8)
 		)
@@
 			(width 0)
 			(type default)
-		)
-	)
-	(hierarchical_label "3V3"
-		(shape input)
-		(at 81.28 58.42 90)
-		(effects
-			(font
-				(size 1.27 1.27)
-			)
-			(justify left)
 		)
 	)
@@
 		(shape input)
 		(at 139.7 83.82 0)
+		(effects
+			(font
+				(size 1.27 1.27)
+			)
+			(justify left)
+		)
+	)
+	(hierarchical_label "PWM_I-"
+		(shape input)
+		(at 139.7 90.17 0)
 		(effects
 			(font
@@
 				(path "/23f2f192-8d8a-4d18-9a9e-f5d6a1224b2d/7e298410-b788-4168-b974-c1c32784a86d"
 					(reference "R10")
+					(unit 1)
+				)
+			)
+		)
+	)
+	(symbol
+		(lib_id "power:GNDREF")
+		(at 135.89 91.44 0)
+		(unit 1)
+		(exclude_from_sim no)
+		(in_bom yes)
+		(on_board yes)
+		(dnp no)
+		(fields_autoplaced yes)
+		(property "Reference" "#PWR017"
+			(at 135.89 97.79 0)
+			(effects
+				(font
+					(size 1.27 1.27)
+				)
+				(hide yes)
+			)
+		)
+		(property "Value" "GNDREF"
+			(at 135.89 96.52 0)
+			(effects
+				(font
+					(size 1.27 1.27)
+				)
+				(hide yes)
+			)
+		)
+		(property "Footprint" ""
+			(at 135.89 91.44 0)
+			(effects
+				(font
+					(size 1.27 1.27)
+				)
+				(hide yes)
+			)
+		)
+		(property "Datasheet" ""
+			(at 135.89 91.44 0)
+			(effects
+				(font
+					(size 1.27 1.27)
+				)
+				(hide yes)
+			)
+		)
+		(property "Description" "Power symbol creates a global label with name \"GNDREF\" , reference supply ground"
+			(at 135.89 91.44 0)
+			(effects
+				(font
+					(size 1.27 1.27)
+				)
+				(hide yes)
+			)
+		)
+		(pin "1"
+		)
+		(instances
+			(project "SolderingStation"
+				(path "/23f2f192-8d8a-4d18-9a9e-f5d6a1224b2d/7e298410-b788-4168-b974-c1c32784a86d"
+					(reference "#PWR017")
 					(unit 1)
 				)
@@
 					(unit 1)
 				)
-			)
-		)
-	)
-	(symbol
-		(lib_id "Device:R")
-		(at 81.28 67.31 0)
-		(unit 1)
-		(exclude_from_sim no)
-		(in_bom yes)
-		(on_board yes)
-		(dnp no)
-		(property "Reference" "R15"
-			(at 82.55 66.04 0)
-			(effects
-				(font
-					(size 1.27 1.27)
-				)
-				(justify left)
-			)
-		)
-		(property "Value" "10k"
-			(at 82.55 68.58 0)
-			(effects
-				(font
-					(size 1.27 1.27)
-				)
-				(justify left)
-			)
-		)
-		(property "Footprint" ""
-			(at 79.502 67.31 90)
-			(effects
-				(font
-					(size 1.27 1.27)
-				)
-				(hide yes)
-			)
-		)
-		(property "Datasheet" "~"
-			(at 81.28 67.31 0)
-			(effects
-				(font
-					(size 1.27 1.27)
-				)
-				(hide yes)
-			)
-		)
-		(property "Description" "Resistor"
-			(at 81.28 67.31 0)
-			(effects
-				(font
-					(size 1.27 1.27)
-				)
-				(hide yes)
-			)
-		)
-		(pin "2"
-		)
-		(pin "1"
-		)
-		(instances
-			(project "SolderingStation"
-				(path "/23f2f192-8d8a-4d18-9a9e-f5d6a1224b2d/7e298410-b788-4168-b974-c1c32784a86d"
-					(reference "R15")
-					(unit 1)
-				)

Commit message: starting pcb
Parts:
- C4: value 10u 35V -> 10uF 50V; footprint (none) -> Capacitor_SMD:C_1206_3216Metric
- D2: footprint Diode_THT:D_DO-35_SOD27_P2.54mm_Vertical_KathodeUp -> Diode_SMD:D_SMA
- Q1: footprint (none) -> Package_TO_SOT_SMD:TO-252-2
- Q2: footprint Package_TO_SOT_THT:TO-92_Inline -> Package_TO_SOT_SMD:SOT-23-3
- R10, R16: footprint (none) -> Resistor_THT:R_Axial_DIN0207_L6.3mm_D2.5mm_P7.62mm_Horizontal
- R11: footprint (none) -> Resistor_SMD:R_0603_1608Metric
Changed lines of the file:
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@@
 			)
 		)
-		(property "Footprint" "Package_TO_SOT_THT:TO-92_Inline"
+		(property "Footprint" "Package_TO_SOT_SMD:SOT-23-3"
 			(at 114.3 75.565 0)
 			(effects
@@
 			)
 		)
-		(property "Footprint" ""
+		(property "Footprint" "Resistor_THT:R_Axial_DIN0207_L6.3mm_D2.5mm_P7.62mm_Horizontal"
 			(at 105.41 60.198 90)
 			(effects
@@
 			)
 		)
-		(property "Value" "10u 35V"
+		(property "Value" "10uF 50V"
 			(at 101.6063 80.01 90)
 			(effects
@@
 			)
 		)
-		(property "Footprint" ""
+		(property "Footprint" "Capacitor_SMD:C_1206_3216Metric"
 			(at 101.6 83.82 0)
 			(effects
@@
 			)
 		)
-		(property "Footprint" ""
+		(property "Footprint" "Resistor_SMD:R_0603_1608Metric"
 			(at 90.17 75.438 90)
 			(effects
@@
 			)
 		)
-		(property "Footprint" ""
+		(property "Footprint" "Package_TO_SOT_SMD:TO-252-2"
 			(at 134.62 55.88 0)
 			(effects
@@
 			)
 		)
-		(property "Footprint" "Diode_THT:D_DO-35_SOD27_P2.54mm_Vertical_KathodeUp"
+		(property "Footprint" "Diode_SMD:D_SMA"
 			(at 105.41 55.245 0)
 			(effects
@@
 			)
 		)
-		(property "Footprint" ""
+		(property "Footprint" "Resistor_THT:R_Axial_DIN0207_L6.3mm_D2.5mm_P7.62mm_Horizontal"
 			(at 105.41 67.818 90)
 			(effects

Commit message: pcb mvp
Parts:
- Q1: value AOD4184 -> IRLZ44N; footprint Package_TO_SOT_SMD:TO-252-2 -> Package_TO_SOT_THT:TO-220-3_Vertical

Commit message: last
Parts:
- C4: value 10uF 50V -> 10uF; LCSC (none) -> C13585
- D2: LCSC (none) -> C22452
- D3: footprint Diode_SMD:D_SOD-123F -> Diode_THT:D_DO-35_SOD27_P2.54mm_Vertical_AnodeUp
- Q2: value S8050 -> 2N2222; footprint Package_TO_SOT_SMD:SOT-23-3 -> Package_TO_SOT_THT:TO-92_Inline; LCSC (none) -> C2146
- R11: footprint Resistor_SMD:R_0603_1608Metric -> Resistor_SMD:R_0805_2012Metric_Pad1.20x1.40mm_HandSolder; LCSC (none) -> C4190
Changed lines of the file:
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@@
 			)
 		)
-		(property "Value" "S8050"
+		(property "Value" "2N2222"
 			(at 113.792 74.93 0)
 			(show_name no)
@@
 			)
 		)
-		(property "Footprint" "Package_TO_SOT_SMD:SOT-23-3"
+		(property "Footprint" "Package_TO_SOT_THT:TO-92_Inline"
 			(at 114.3 75.565 0)
 			(hide yes)
@@
 		)
 		(property "Description" "0.7A Ic, 20V Vce, Low Voltage High Current NPN Transistor, TO-92"
+			(at 109.22 73.66 0)
+			(hide yes)
+			(show_name no)
+			(do_not_autoplace no)
+			(effects
+				(font
+					(size 1.27 1.27)
+				)
+			)
+		)
+		(property "LCSC" "C2146"
 			(at 109.22 73.66 0)
 			(hide yes)
@@
 		(property "Description" "Resistor"
 			(at 105.41 58.42 0)
+			(hide yes)
+			(show_name no)
+			(do_not_autoplace no)
+			(effects
+				(font
+					(size 1.27 1.27)
+				)
+			)
+		)
+		(property "LCSC" ""
+			(at 105.41 58.42 90)
 			(hide yes)
 			(show_name no)
@@
 			)
 		)
-		(property "Value" "10uF 50V"
+		(property "Value" "10uF"
 			(at 101.6063 80.01 90)
 			(show_name no)
@@
 		(property "Description" "Unpolarized capacitor, small symbol"
 			(at 101.6 83.82 0)
+			(hide yes)
+			(show_name no)
+			(do_not_autoplace no)
+			(effects
+				(font
+					(size 1.27 1.27)
+				)
+			)
+		)
+		(property "LCSC" "C13585"
+			(at 101.6 83.82 90)
 			(hide yes)
 			(show_name no)
@@
 			)
 		)
-		(property "Footprint" "Diode_SMD:D_SOD-123F"
+		(property "Footprint" "Diode_THT:D_DO-35_SOD27_P2.54mm_Vertical_AnodeUp"
 			(at 117.475 74.93 0)
 			(hide yes)
@@
 		(property "Description" "500mW Zener Diode, SOD-123F"
 			(at 121.92 74.93 0)
+			(hide yes)
+			(show_name no)
+			(do_not_autoplace no)
+			(effects
+				(font
+					(size 1.27 1.27)
+				)
+			)
+		)
+		(property "LCSC" ""
+			(at 121.92 74.93 90)
 			(hide yes)
 			(show_name no)
@@
 			)
 		)
-		(property "Footprint" "Resistor_SMD:R_0603_1608Metric"
+		(property "Footprint" "Resistor_SMD:R_0805_2012Metric_Pad1.20x1.40mm_HandSolder"
 			(at 90.17 75.438 90)
 			(hide yes)
@@
 		(property "Description" "Resistor"
 			(at 90.17 73.66 0)
+			(hide yes)
+			(show_name no)
+			(do_not_autoplace no)
+			(effects
+				(font
+					(size 1.27 1.27)
+				)
+			)
+		)
+		(property "LCSC" "C4190"
+			(at 90.17 73.66 90)
 			(hide yes)
 			(show_name no)
@@
 			)
 		)
+		(property "LCSC" ""
+			(at 129.54 58.42 0)
+			(hide yes)
+			(show_name no)
+			(do_not_autoplace no)
+			(effects
+				(font
+					(size 1.27 1.27)
+				)
+			)
+		)
 		(pin "3"
 		)
@@
 			)
 		)
+		(property "LCSC" "C22452"
+			(at 105.41 50.8 0)
+			(hide yes)
+			(show_name no)
+			(do_not_autoplace no)
+			(effects
+				(font
+					(size 1.27 1.27)
+				)
+			)
+		)
 		(pin "1"
 		)
@@
 			(hide yes)
 			(show_name no)
+			(do_not_autoplace no)
+			(effects
+				(font
+					(size 1.27 1.27)
+				)
+			)
+		)
+		(property "LCSC" ""
+			(at 105.41 66.04 90)
+			(hide yes)
+			(show_name no)
