File: hardware/MUG.kicad_sch (KiCad schematic)
At the start: 33 parts, among them Q5 2N2222, SW1 SW_SPST, U5 STM32F103C8Tx, Y1 X50328MSB2GI

Commit message: fast
Connections:
- net SCL: now also U5.45 (PB8); no longer U5.42 (PB6)
- net SDA: now also U5.46 (PB9); no longer U5.43 (PB7)
- net at R31.1: now also U5.42 (PB6); no longer U5.45 (PB8)
- net at R32.1: now also U5.43 (PB7); no longer U5.46 (PB9)
Changed lines of the file:
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@@
-	)
-	(junction
-		(at 27.94 78.74)
-		(diameter 0)
-		(color 0 0 0 0)
 	)
 	(junction
@@
 	)
 	(junction
-		(at 115.57 66.04)
+		(at 27.94 83.82)
 		(diameter 0)
 		(color 0 0 0 0)
 	)
 	(junction
-		(at 35.56 76.2)
+		(at 35.56 81.28)
+		(diameter 0)
+		(color 0 0 0 0)
+	)
+	(junction
+		(at 115.57 66.04)
 		(diameter 0)
 		(color 0 0 0 0)
@@
 	(wire
 		(pts
-			(xy 27.94 78.74) (xy 77.47 78.74)
-		)
-		(stroke
-			(width 0)
-			(type default)
-		)
-	)
-	(wire
-		(pts
 			(xy 90.17 25.4) (xy 90.17 19.05)
 		)
@@
 	(wire
 		(pts
+			(xy 27.94 83.82) (xy 77.47 83.82)
+		)
+		(stroke
+			(width 0)
+			(type default)
+		)
+	)
+	(wire
+		(pts
 			(xy 113.03 48.26) (xy 115.57 48.26)
 		)
@@
 	(wire
 		(pts
-			(xy 64.77 83.82) (xy 67.31 83.82)
-		)
-		(stroke
-			(width 0)
-			(type default)
-		)
-	)
-	(wire
-		(pts
-			(xy 27.94 72.39) (xy 27.94 78.74)
+			(xy 64.77 78.74) (xy 67.31 78.74)
 		)
 		(stroke
@@
 	(wire
 		(pts
-			(xy 35.56 76.2) (xy 77.47 76.2)
-		)
-		(stroke
-			(width 0)
-			(type default)
-		)
-	)
-	(wire
-		(pts
 			(xy 171.45 40.64) (xy 171.45 44.45)
 		)
@@
 	(wire
 		(pts
-			(xy 24.13 76.2) (xy 35.56 76.2)
-		)
-		(stroke
-			(width 0)
-			(type default)
-		)
-	)
-	(wire
-		(pts
-			(xy 64.77 81.28) (xy 67.31 81.28)
+			(xy 24.13 81.28) (xy 35.56 81.28)
+		)
+		(stroke
+			(width 0)
+			(type default)
+		)
+	)
+	(wire
+		(pts
+			(xy 64.77 76.2) (xy 67.31 76.2)
 		)
 		(stroke
@@
 	(wire
 		(pts
-			(xy 74.93 83.82) (xy 77.47 83.82)
-		)
-		(stroke
-			(width 0)
-			(type default)
-		)
-	)
-	(wire
-		(pts
 			(xy 115.57 50.8) (xy 115.57 53.34)
 		)
@@
 	(wire
 		(pts
+			(xy 27.94 72.39) (xy 27.94 83.82)
+		)
+		(stroke
+			(width 0)
+			(type default)
+		)
+	)
+	(wire
+		(pts
 			(xy 161.29 88.9) (xy 161.29 82.55)
 		)
@@
 	(wire
 		(pts
-			(xy 35.56 72.39) (xy 35.56 76.2)
+			(xy 35.56 72.39) (xy 35.56 81.28)
 		)
 		(stroke
@@
 	(wire
 		(pts
+			(xy 35.56 81.28) (xy 77.47 81.28)
+		)
+		(stroke
+			(width 0)
+			(type default)
+		)
+	)
+	(wire
+		(pts
 			(xy 115.57 66.04) (xy 125.73 66.04)
 		)
@@
 	(wire
 		(pts
+			(xy 74.93 76.2) (xy 77.47 76.2)
+		)
+		(stroke
+			(width 0)
+			(type default)
+		)
+	)
+	(wire
+		(pts
 			(xy 190.5 40.64) (xy 190.5 44.45)
 		)
@@
 	(wire
 		(pts
-			(xy 24.13 78.74) (xy 27.94 78.74)
+			(xy 24.13 83.82) (xy 27.94 83.82)
 		)
 		(stroke
@@
 	(wire
 		(pts
-			(xy 74.93 81.28) (xy 77.47 81.28)
-		)
-		(stroke
-			(width 0)
-			(type default)
-		)
-	)
-	(wire
-		(pts
 			(xy 69.85 54.61) (xy 69.85 55.88)
 		)
@@
 		(pts
 			(xy 74.93 93.98) (xy 77.47 93.98)
+		)
+		(stroke
+			(width 0)
+			(type default)
+		)
+	)
+	(wire
+		(pts
+			(xy 74.93 78.74) (xy 77.47 78.74)
 		)
 		(stroke
@@
 	(hierarchical_label "SDA"
 		(shape input)
-		(at 24.13 78.74 180)
+		(at 24.13 83.82 180)
 		(effects
 			(font
@@
 	(hierarchical_label "A_EC_S2"
 		(shape input)
-		(at 64.77 83.82 180)
+		(at 64.77 78.74 180)
 		(effects
 			(font
@@
 	(hierarchical_label "A_EC_S1"
 		(shape input)
-		(at 64.77 81.28 180)
+		(at 64.77 76.2 180)
 		(effects
 			(font
@@
 	(hierarchical_label "SCL"
 		(shape input)
-		(at 24.13 76.2 180)
+		(at 24.13 81.28 180)
 		(effects
 			(font
@@
 	(symbol
 		(lib_id "Device:R")
-		(at 71.12 81.28 270)
+		(at 71.12 76.2 270)
 		(unit 1)
 		(body_style 1)
@@
 		(dnp no)
 		(property "Reference" "R31"
+			(at 71.12 71.12 90)
+			(hide yes)
+			(show_name no)
+			(do_not_autoplace no)
+			(effects
+				(font
+					(size 1.27 1.27)
+				)
+			)
+		)
+		(property "Value" "1k"
 			(at 71.12 76.2 90)
-			(hide yes)
-			(show_name no)
-			(do_not_autoplace no)
-			(effects
-				(font
-					(size 1.27 1.27)
-				)
-			)
-		)
-		(property "Value" "1k"
-			(at 71.12 81.28 90)
 			(show_name no)
 			(do_not_autoplace no)
@@
 		)
 		(property "Footprint" "Resistor_SMD:R_0805_2012Metric_Pad1.20x1.40mm_HandSolder"
-			(at 71.12 79.502 90)
+			(at 71.12 74.422 90)
 			(hide yes)
 			(show_name no)
@@
 		)
 		(property "Datasheet" ""
-			(at 71.12 81.28 0)
+			(at 71.12 76.2 0)
 			(hide yes)
 			(show_name no)
@@
 		)
 		(property "Description" "Resistor"
-			(at 71.12 81.28 0)
+			(at 71.12 76.2 0)
 			(hide yes)
 			(show_name no)
@@
 		)
 		(property "LCSC" "C21190"
-			(at 71.12 81.28 90)
+			(at 71.12 76.2 90)
 			(hide yes)
 			(show_name no)
@@
 	(symbol
 		(lib_id "Device:R")
-		(at 71.12 83.82 270)
+		(at 71.12 78.74 270)
 		(unit 1)
 		(body_style 1)
@@
 		(dnp no)
 		(property "Reference" "R32"
+			(at 71.12 73.66 90)
+			(hide yes)
+			(show_name no)
+			(do_not_autoplace no)
+			(effects
+				(font
+					(size 1.27 1.27)
+				)
+			)
+		)
+		(property "Value" "1k"
 			(at 71.12 78.74 90)
-			(hide yes)
-			(show_name no)
-			(do_not_autoplace no)
-			(effects
-				(font
-					(size 1.27 1.27)
-				)
-			)
-		)
-		(property "Value" "1k"
-			(at 71.12 83.82 90)
 			(show_name no)
 			(do_not_autoplace no)
@@
 		)
 		(property "Footprint" "Resistor_SMD:R_0805_2012Metric_Pad1.20x1.40mm_HandSolder"
-			(at 71.12 82.042 90)
+			(at 71.12 76.962 90)
 			(hide yes)
 			(show_name no)
@@
 		)
 		(property "Datasheet" ""
-			(at 71.12 83.82 0)
+			(at 71.12 78.74 0)
 			(hide yes)
 			(show_name no)
@@
 		)
 		(property "Description" "Resistor"
-			(at 71.12 83.82 0)
+			(at 71.12 78.74 0)
 			(hide yes)
 			(show_name no)
@@
 		)
 		(property "LCSC" "C21190"
-			(at 71.12 83.82 90)
-			(hide yes)
-			(show_name no)
+			(at 71.12 78.74 90)
+			(hide yes)
+			(show_name no)
